File: NightController/NightController.kicad_pcb (KiCad board)
At the start: 2 copper layers, 9.8 x 2.8 mm, 214 parts, among them J201 Conn_02x20_Odd_Even, J202 Conn_02x20_Odd_Even, U301 LP5036, U302 LP5036, U303 LP5036, U304 LP5036

Commit message: working on LED PCB
Parts:
- removed the C303 at (55.7, 63.5)
- removed C304: 1uF 50V, Capacitor_SMD:C_0603_1608Metric_Pad1.08x0.95mm_HandSolder
- removed D301, D302, D303, D304, D305, D306, D307, D308, D309, D310, D311, D312, D313, D314, D315, D316, D317, D318, D319, D320, D321, D322, D323, D324, D325, D326, D327, D328, D329, D330, D331, D332, D333, D334, D335, D336, D337, D338, D339, D340, D341, D342, D343, D344, D345, D346, D347, D348: SMLVN6RGB, LED_SMD:LED_ROHM_SMLVN6
- removed the R302 at (55.1, 20.0)
- removed R305, R379, R380, R381, R383: R, Resistor_SMD:R_0402_1005Metric_Pad0.72x0.64mm_HandSolder
- removed R306, R382, R384: 10k 5%, Resistor_SMD:R_0402_1005Metric_Pad0.72x0.64mm_HandSolder
- removed R307, R308, R309, R310, R311, R312, R313, R314, R315, R316, R317, R318, R319, R320, R321, R322, R323, R324, R325, R326, R327, R328, R329, R330, R331, R332, R333, R334, R335, R336, R337, R338, R339, R340, R341, R342, R343, R344, R345, R346, R347, R348, R349, R350, R351, R352, R353, R354, R355, R356, R357, R358, R359, R360, R361, R362, R363, R364, R365, R366, R367, R368, R369, R370, R371, R372, R373, R374, R375, R376, R377, R378, R385, R386, R387, R388, R389, R390, R391, R392, R393, R394, R395, R396, R397, R398, R399, R400, R401, R402, R403, R404, R405, R406, R407, R408, R409, R410, R411, R412, R413, R414, R415, R416, R417, R418, R419, R420, R421, R422, R423, R424, R425, R426, R427, R428, R429, R430, R431, R432, R433, R434, R435, R436, R437, R438, R439, R440, R441, R442, R443, R444, R445, R446, R447, R448, R449, R450, R451, R452, R453, R454, R455, R456: 1k 5%, Resistor_SMD:R_0402_1005Metric_Pad0.72x0.64mm_HandSolder
- added C301: 4.7uF 25V, Capacitor_SMD:C_0402_1005Metric_Pad0.74x0.62mm_HandSolder, B.Cu at (155.8, 98.7)
- added FID101: Fiducial, Fiducial:Fiducial_0.5mm_Mask1mm, F.Cu at (132.0, 110.0)
- added FID102: Fiducial, Fiducial:Fiducial_0.5mm_Mask1mm, B.Cu at (168.0, 90.0)
- added FID103: Fiducial, Fiducial:Fiducial_0.5mm_Mask1mm, F.Cu at (161.0, 117.0)
- added FID104: Fiducial, Fiducial:Fiducial_0.5mm_Mask1mm, B.Cu at (168.0, 110.0)
- added FID105: Fiducial, Fiducial:Fiducial_0.5mm_Mask1mm, F.Cu at (139.0, 83.0)
- added FID106: Fiducial, Fiducial:Fiducial_0.5mm_Mask1mm, B.Cu at (139.0, 117.0)
- added H101: MountingHole_Pad, MountingHole:MountingHole_3.2mm_M3_Pad_Via, F.Cu at (135.0, 86.0)
- added H102: MountingHole_Pad, MountingHole:MountingHole_3.2mm_M3_Pad_Via, F.Cu at (135.0, 114.0)
- added H103: MountingHole_Pad, MountingHole:MountingHole_3.2mm_M3_Pad_Via, F.Cu at (165.0, 114.0)
- added H104: MountingHole_Pad, MountingHole:MountingHole_3.2mm_M3_Pad_Via, F.Cu at (165.0, 86.0)
- added TP301: TestPoint_Small, TestPoint:TestPoint_Loop_D1.80mm_Drill1.0mm_Beaded, F.Cu at (167.5, 102.5)
- added TP302: TestPoint_Small, TestPoint:TestPoint_Loop_D1.80mm_Drill1.0mm_Beaded, F.Cu at (167.5, 97.5)
- added TP303: TestPoint_Small, TestPoint:TestPoint_Loop_D1.80mm_Drill1.0mm_Beaded, F.Cu at (167.5, 92.5)
- added TP304: TestPoint_Small, TestPoint:TestPoint_Loop_D1.80mm_Drill1.0mm_Beaded, F.Cu at (167.5, 107.5)
- added TP305: TestPoint_Small, TestPoint:TestPoint_Loop_D1.80mm_Drill1.0mm_Beaded, F.Cu at (157.5, 115.0)
- added TP306: TestPoint_Small, TestPoint:TestPoint_Loop_D1.80mm_Drill1.0mm_Beaded, F.Cu at (152.5, 115.0)
- added U305: EAST1410RGBW02, EAST1410RGBW02:SMD_EAST1410RGBW02_EVE, F.Cu at (140.0, 110.0)
- added U306: EAST1410RGBW02, EAST1410RGBW02:SMD_EAST1410RGBW02_EVE, F.Cu at (140.0, 100.0)
- added U307: EAST1410RGBW02, EAST1410RGBW02:SMD_EAST1410RGBW02_EVE, F.Cu at (140.0, 90.0)
- added U308: EAST1410RGBW02, EAST1410RGBW02:SMD_EAST1410RGBW02_EVE, F.Cu at (150.0, 90.0)
- added U309: EAST1410RGBW02, EAST1410RGBW02:SMD_EAST1410RGBW02_EVE, F.Cu at (160.0, 90.0)
- added U310: EAST1410RGBW02, EAST1410RGBW02:SMD_EAST1410RGBW02_EVE, F.Cu at (160.0, 100.0)
- C302: value 1uF 50V -> 100nF 50V; footprint Capacitor_SMD:C_0603_1608Metric_Pad1.08x0.95mm_HandSolder -> Capacitor_SMD:C_0402_1005Metric_Pad0.74x0.62mm_HandSolder; moved to B.Cu
- C303: renamed from C301; footprint Capacitor_SMD:C_0603_1608Metric_Pad1.08x0.95mm_HandSolder -> Capacitor_SMD:C_0402_1005Metric_Pad0.74x0.62mm_HandSolder; moved to B.Cu
- J201, J202: footprint Connector_Molex:Molex_SlimStack_502426-4010_2x20_P0.40mm_Vertical -> Connector_Molex:Molex_SlimStack_54722-0404_2x20_P0.50mm_Vertical; moved to B.Cu
- R301: value R -> 0E 5%; moved to B.Cu
- R302: renamed from R303; value R -> 0E 5%; moved to B.Cu
- R303: renamed from R304; moved to B.Cu
- U302, U303, U304: value LP5036 -> EAST1410RGBW02; footprint Package_DFN_QFN:VQFN-46-1EP_5x6mm_P0.4mm_EP2.8x3.8mm -> EAST1410RGBW02:SMD_EAST1410RGBW02_EVE
- moved J202 138.8 mm to (160.0, 100.0), turned to 90 degrees
- moved R303 128.0 mm to (154.7, 104.4), turned to -90 degrees
- moved R301 125.5 mm to (153.8, 95.7), turned to 90 degrees
- moved R302 124.1 mm to (155.0, 95.7), turned to 90 degrees
- moved J201 120.2 mm to (140.0, 100.0), turned to 90 degrees
- moved C303 108.2 mm to (153.7, 104.4), turned to -90 degrees
- moved C302 106.0 mm to (154.8, 98.7), turned to 90 degrees
- moved U303 105.0 mm to (160.0, 110.0), turned to 90 degrees
- moved U302 97.6 mm to (150.0, 100.0)
- moved U304 90.4 mm to (150.0, 110.0), turned to 90 degrees
- moved U301 36.8 mm to (150.0, 100.0)
Connections:
- C302 pad 1: Net-(U302-VCAP) -> +5V
- J201 pad 12: LP_EN -> unconnected-(J201-Pin_12-Pad12)
- J201 pad 14: LP_SCL -> unconnected-(J201-Pin_14-Pad14)
- J201 pad 16: LP_SDA -> unconnected-(J201-Pin_16-Pad16)
- J202 pad 12: LP_EN -> /Connectors/LP_EN
- J202 pad 14: LP_SCL -> /Connectors/LP_SCL
- J202 pad 16: LP_SDA -> /Connectors/LP_SDA
- U301 pad 1: Net-(D301-GK) -> Net-(U301-OUT0)
- U301 pad 10: Net-(D307-GK) -> Net-(U301-OUT9)
- U301 pad 11: Net-(D307-RK) -> Net-(U301-OUT10)
- U301 pad 12: Net-(D307-BK) -> Net-(U301-OUT11)
- U301 pad 2: Net-(D301-RK) -> Net-(U301-OUT1)
- U301 pad 3: Net-(D301-BK) -> Net-(U301-OUT2)
- U301 pad 4: Net-(D303-GK) -> Net-(U301-OUT3)
- U301 pad 40: unconnected-(U301-VCC-Pad40) -> +5V
- U301 pad 41: LP_SDA -> /Connectors/LP_SDA
- U301 pad 42: LP_SCL -> /Connectors/LP_SCL
- U301 pad 43: LP_EN -> /Connectors/LP_EN
- U301 pad 5: Net-(D303-RK) -> Net-(U301-OUT4)
- U301 pad 6: Net-(D303-BK) -> Net-(U301-OUT5)
- U301 pad 7: Net-(D305-GK) -> Net-(U301-OUT6)
- U301 pad 8: Net-(D305-RK) -> Net-(U301-OUT7)
- U301 pad 9: Net-(D305-BK) -> Net-(U301-OUT8)
- U302 pad 1: Net-(D302-GK) -> +5V
- U302 pad 2: Net-(D302-RK) -> Net-(U301-OUT0)
- U302 pad 3: Net-(D302-BK) -> Net-(U301-OUT1)
- U302 pad 4: Net-(D304-GK) -> Net-(U301-OUT2)
- U302 pad 5: Net-(D304-RK) -> Net-(U301-OUT3)
- U302 pad 6: Net-(D304-BK) -> unconnected-(U302-Pad6)
- U303 pad 1: Net-(D325-GK) -> +5V
- U303 pad 2: Net-(D325-RK) -> Net-(U301-OUT4)
- U303 pad 3: Net-(D325-BK) -> Net-(U301-OUT5)
- U303 pad 4: Net-(D327-GK) -> Net-(U301-OUT6)
- U303 pad 5: Net-(D327-RK) -> Net-(U301-OUT7)
- U303 pad 6: Net-(D327-BK) -> unconnected-(U303-Pad6)
- U304 pad 1: Net-(D326-GK) -> +5V
- U304 pad 2: Net-(D326-RK) -> Net-(U301-OUT8)
- U304 pad 3: Net-(D326-BK) -> Net-(U301-OUT9)
- U304 pad 4: Net-(D328-GK) -> Net-(U301-OUT10)
- U304 pad 5: Net-(D328-RK) -> Net-(U301-OUT11)
- U304 pad 6: Net-(D328-BK) -> unconnected-(U304-Pad6)
Routing:
- net +3V3: track 0.00 -> 57.3 mm, vias 0 -> 8
- net GND: track 0.00 -> 50.0 mm, vias 0 -> 29
- net /Connectors/LP_SDA: track 0.00 -> 21.4 mm, vias 0 -> 1
- net /Connectors/LP_SCL: track 0.00 -> 20.8 mm, vias 0 -> 1
- net /Connectors/LP_EN: track 0.00 -> 19.6 mm, vias 0 -> 1
- net Net-(U301-OUT5): track 0.00 -> 17.5 mm, vias 0 -> 1
- net Net-(U301-OUT30): track 1.51 -> 18.2 mm
- net Net-(U301-OUT6): track 0.00 -> 16.3 mm, vias 0 -> 1
- net Net-(U301-OUT4): track 0.00 -> 15.8 mm, vias 0 -> 1
- net Net-(U301-OUT7): track 0.00 -> 15.8 mm, vias 0 -> 1
- net Net-(U301-OUT31): track 1.54 -> 17.2 mm
- net Net-(U301-OUT29): track 1.51 -> 16.0 mm
- net Net-(U301-OUT12): track 1.57 -> 15.4 mm
- net Net-(U301-OUT28): track 1.54 -> 15.2 mm
- net Net-(U301-OUT33): track 1.51 -> 15.0 mm
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- added copper zone on In1.Cu, net +5V
- added copper zone on In2.Cu, net GND
Other:
- board size 9.8 x 2.8 mm -> 40 x 38 mm
- copper layers 2 -> 4

Commit message: Update NightController.kicad_pcb
Other:
- board text added: "+5V"
- board text added: "CONN1"
- board text added: "CONN2"
- board text added: "EN"
- board text added: "GND"
- board text added: "JLCJLCJLCJLC"
- board text added: "NightLight LED Board"
- board text added: "SCL"
- board text added: "SDA"

Commit message: Finisched digital one
Parts:
- removed R301, R302: 0E 5%, Resistor_SMD:R_0402_1005Metric_Pad0.72x0.64mm_HandSolder
- removed R303: 10k 5%, Resistor_SMD:R_0402_1005Metric_Pad0.72x0.64mm_HandSolder
- removed U301: LP5036, Package_DFN_QFN:VQFN-46-1EP_5x6mm_P0.4mm_EP2.8x3.8mm
- removed U302, U303, U304, U305, U306, U307, U308, U309, U310: EAST1410RGBW02, EAST1410RGBW02:SMD_EAST1410RGBW02_EVE
- added C304: C, Capacitor_SMD:C_0402_1005Metric_Pad0.74x0.62mm_HandSolder, F.Cu at (140.4, 98.0)
- added C305: C, Capacitor_SMD:C_0402_1005Metric_Pad0.74x0.62mm_HandSolder, F.Cu at (139.7, 111.8)
- added C306: C, Capacitor_SMD:C_0402_1005Metric_Pad0.74x0.62mm_HandSolder, F.Cu at (149.7, 111.8)
- added C307: C, Capacitor_SMD:C_0402_1005Metric_Pad0.74x0.62mm_HandSolder, F.Cu at (159.7, 111.8)
- added C308: C, Capacitor_SMD:C_0402_1005Metric_Pad0.74x0.62mm_HandSolder, F.Cu at (160.4, 98.0)
- added C309: C, Capacitor_SMD:C_0402_1005Metric_Pad0.74x0.62mm_HandSolder, F.Cu at (152.2, 101.8)
- added C310: C, Capacitor_SMD:C_0402_1005Metric_Pad0.74x0.62mm_HandSolder, F.Cu at (147.2, 101.8)
- added D301: SK6805, LED_SMD:LED_SK6805_PLCC4_2.4x2.7mm_P1.3mm, F.Cu at (160.0, 90.0)
- added D302: SK6805, LED_SMD:LED_SK6805_PLCC4_2.4x2.7mm_P1.3mm, F.Cu at (150.0, 90.0)
- added D303: SK6805, LED_SMD:LED_SK6805_PLCC4_2.4x2.7mm_P1.3mm, F.Cu at (140.0, 90.0)
- added D304: SK6805, LED_SMD:LED_SK6805_PLCC4_2.4x2.7mm_P1.3mm, F.Cu at (140.0, 100.0)
- added D305: SK6805, LED_SMD:LED_SK6805_PLCC4_2.4x2.7mm_P1.3mm, F.Cu at (140.1, 109.8)
- added D306: SK6805, LED_SMD:LED_SK6805_PLCC4_2.4x2.7mm_P1.3mm, F.Cu at (150.1, 109.8)
- added D307: SK6805, LED_SMD:LED_SK6805_PLCC4_2.4x2.7mm_P1.3mm, F.Cu at (160.1, 109.8)
- added D308: SK6805, LED_SMD:LED_SK6805_PLCC4_2.4x2.7mm_P1.3mm, F.Cu at (160.0, 100.0)
- added D309: SK6805, LED_SMD:LED_SK6805_PLCC4_2.4x2.7mm_P1.3mm, F.Cu at (147.5, 100.0)
- added D310: SK6805, LED_SMD:LED_SK6805_PLCC4_2.4x2.7mm_P1.3mm, F.Cu at (152.5, 100.0)
- C301: value 4.7uF 25V -> C; moved to F.Cu
- C302: value 100nF 50V -> C; moved to F.Cu
- C303: value 1uF 50V -> C; moved to F.Cu
- moved TP303 27.0 mm to (152.5, 115.0)
- moved TP306 27.0 mm to (167.5, 92.5)
- moved C303 21.1 mm to (140.4, 88.0), turned to 180 degrees
- moved TP302 20.2 mm to (157.5, 115.0)
- moved TP305 20.2 mm to (167.5, 97.5)
- moved C301 11.7 mm to (160.4, 88.0), turned to 180 degrees
- moved C302 11.5 mm to (150.4, 88.0), turned to 180 degrees
- moved TP301 5.00 mm to (167.5, 107.5)
- moved TP304 5.00 mm to (167.5, 102.5)
Connections:
- C303 pad 1: Net-(U301-VCAP) -> +5V
- J202 pad 12: /Connectors/LP_EN -> unconnected-(J202-Pin_12-Pad12)
- J202 pad 14: /Connectors/LP_SCL -> unconnected-(J202-Pin_14-Pad14)
- J202 pad 16: /Connectors/LP_SDA -> unconnected-(J202-Pin_16-Pad16)
- J202 pad 27: unconnected-(J202-Pin_27-Pad27) -> /Connectors/DOUT
- J202 pad 29: unconnected-(J202-Pin_29-Pad29) -> /Connectors/DIN
- TP301 pad 1: /Connectors/LP_EN -> GND
- TP302 pad 1: /Connectors/LP_SCL -> +5V
- TP303 pad 1: /Connectors/LP_SDA -> GND
- TP304 pad 1: GND -> +5V
- TP305 pad 1: +5V -> /Connectors/DOUT
- TP306 pad 1: GND -> /Connectors/DIN
Routing:
- net /Connectors/LP_SDA: track 21.4 -> 0.00 mm, vias 1 -> 0
- net /Connectors/LP_SCL: track 20.8 -> 0.00 mm, vias 1 -> 0
- net /Connectors/DOUT: track 0.00 -> 20.4 mm
- net /Connectors/LP_EN: track 19.6 -> 0.00 mm, vias 1 -> 0
- net Net-(U301-OUT30): track 18.2 -> 0.00 mm, vias 1 -> 0
- net Net-(U301-OUT5): track 17.5 -> 0.00 mm, vias 1 -> 0
- net +5V: track 43.0 -> 60.4 mm
- net Net-(U301-OUT31): track 17.2 -> 0.00 mm, vias 1 -> 0
- net Net-(U301-OUT6): track 16.3 -> 0.00 mm, vias 1 -> 0
- net Net-(U301-OUT29): track 16.0 -> 0.00 mm, vias 1 -> 0
- net Net-(U301-OUT4): track 15.8 -> 0.00 mm, vias 1 -> 0
- net Net-(U301-OUT7): track 15.8 -> 0.00 mm, vias 1 -> 0
- net /Connectors/DIN: track 0.00 -> 15.7 mm
- net /LED Controller/DO8: track 0.00 -> 15.5 mm
- net Net-(U301-OUT12): track 15.4 -> 0.00 mm, vias 1 -> 0
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Other:
- board text added: "DIN"
- board text added: "DOUT"
- board text removed: "EN"
- board text removed: "SCL"
- board text removed: "SDA"
