File: NightController/NightController.kicad_sch (KiCad schematic)
At the start: 0 parts

Commit message: Working on files
Parts:
- added FID101, FID102, FID103, FID104, FID105, FID106: Fiducial, symbol Mechanical:Fiducial
- added H101, H102, H103, H104: MountingHole_Pad, symbol Mechanical:MountingHole_Pad
Connections:
- new net GND: H101.1, H102.1, H103.1, H104.1
- no-connect marks 0 -> 6
Other:
- sheet Connectors ports: added LP_EN, LP_SCL, LP_SDA; removed none
- sheet LED Controller ports: added LP_EN, LP_SCL, LP_SDA; removed none
- note added: "Mounting holes and fiducials for production"
- title: (none) -> NightLight

Commit message: working on LED PCB
Parts:
- FID101, FID102, FID103, FID104, FID105, FID106: footprint (none) -> Fiducial:Fiducial_0.5mm_Mask1mm
- H101, H102, H103, H104: footprint (none) -> MountingHole:MountingHole_3.2mm_M3_Pad_Via
Changed lines of the file:
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@@
 			)
 		)
-		(property "Footprint" ""
+		(property "Footprint" "Fiducial:Fiducial_0.5mm_Mask1mm"
 			(at 76.2 177.8 0)
 			(effects
@@
 			)
 		)
-		(property "Footprint" ""
+		(property "Footprint" "MountingHole:MountingHole_3.2mm_M3_Pad_Via"
 			(at 39.37 165.1 0)
 			(effects
@@
 			)
 		)
-		(property "Footprint" ""
+		(property "Footprint" "Fiducial:Fiducial_0.5mm_Mask1mm"
 			(at 101.6 165.1 0)
 			(effects
@@
 			)
 		)
-		(property "Footprint" ""
+		(property "Footprint" "Fiducial:Fiducial_0.5mm_Mask1mm"
 			(at 76.2 152.4 0)
 			(effects
@@
 			)
 		)
-		(property "Footprint" ""
+		(property "Footprint" "Fiducial:Fiducial_0.5mm_Mask1mm"
 			(at 76.2 165.1 0)
 			(effects
@@
 			)
 		)
-		(property "Footprint" ""
+		(property "Footprint" "MountingHole:MountingHole_3.2mm_M3_Pad_Via"
 			(at 39.37 190.5 0)
 			(effects
@@
 			)
 		)
-		(property "Footprint" ""
+		(property "Footprint" "MountingHole:MountingHole_3.2mm_M3_Pad_Via"
 			(at 39.37 152.4 0)
 			(effects
@@
 			)
 		)
-		(property "Footprint" ""
+		(property "Footprint" "Fiducial:Fiducial_0.5mm_Mask1mm"
 			(at 101.6 177.8 0)
 			(effects
@@
 			)
 		)
-		(property "Footprint" ""
+		(property "Footprint" "MountingHole:MountingHole_3.2mm_M3_Pad_Via"
 			(at 39.37 177.8 0)
 			(effects
@@
 			)
 		)
-		(property "Footprint" ""
+		(property "Footprint" "Fiducial:Fiducial_0.5mm_Mask1mm"
 			(at 101.6 152.4 0)
 			(effects

Commit message: Finisched digital one
Other:
- sheet Connectors ports: added DIN, DOUT; removed LP_EN, LP_SCL, LP_SDA
- sheet LED Controller ports: added DIN, DOUT; removed LP_EN, LP_SCL, LP_SDA
Changed lines of the file:
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@@
-	(wire
-		(pts
-			(xy 114.3 92.71) (xy 152.4 92.71)
-		)
-		(stroke
-			(width 0)
-			(type default)
-		)
-	)
 	(wire
 		(pts
@@
 			)
 		)
-		(pin "LP_EN" output
-			(at 152.4 92.71 180)
-			(effects
-				(font
-					(size 1.27 1.27)
-				)
-				(justify left)
-			)
-		)
-		(pin "LP_SCL" bidirectional
+		(pin "DOUT" input
 			(at 152.4 106.68 180)
 			(effects
@@
 			)
 		)
-		(pin "LP_SDA" bidirectional
+		(pin "DIN" output
 			(at 152.4 110.49 180)
 			(effects
@@
 			)
 		)
-		(pin "LP_EN" input
-			(at 114.3 92.71 0)
+		(pin "DIN" input
+			(at 114.3 110.49 0)
 			(effects
 				(font
@@
 			)
 		)
-		(pin "LP_SCL" bidirectional
+		(pin "DOUT" output
 			(at 114.3 106.68 0)
 			(effects
 				(font
-					(size 1.27 1.27)
-				)
-				(justify right)
-			)
-		)
-		(pin "LP_SDA" bidirectional
-			(at 114.3 110.49 0)
-			(effects
-				(font
