File: NightController/led_controller.kicad_sch (KiCad schematic)
At the start: 212 parts, among them U401 LP5036, U402 LP5036, U403 LP5036, U404 LP5036

Commit message: Add LED lib
Parts:
- removed C401, C403, C404: 1uF 50V, symbol Device:C
- removed D413, D414, D415, D416, D417, D418, D419, D420, D421, D422, D423, D424, D425, D426, D427, D428, D429, D430, D431, D432, D433, D434, D435, D436, D437, D438, D439, D440, D441, D442, D443, D444, D445, D446, D447, D448: SMLVN6RGB, LED_SMD:LED_ROHM_SMLVN6, symbol LED:SMLVN6RGB
- removed R442, R445, R484, R485, R524, R526: R, symbol Device:R
- removed R446, R487, R528: 10k 5%, symbol Device:R
- removed R447, R448, R449, R450, R451, R452, R453, R454, R455, R456, R457, R458, R459, R460, R461, R462, R463, R464, R465, R466, R467, R468, R469, R470, R471, R472, R473, R474, R475, R476, R477, R478, R479, R480, R481, R482, R488, R489, R490, R491, R492, R493, R494, R495, R496, R497, R498, R499, R500, R501, R502, R503, R504, R505, R506, R507, R508, R509, R510, R511, R512, R513, R514, R515, R516, R517, R518, R519, R520, R521, R522, R523, R529, R530, R531, R532, R533, R534, R535, R536, R537, R538, R539, R540, R541, R542, R543, R544, R545, R546, R547, R548, R549, R550, R551, R552, R553, R554, R555, R556, R557, R558, R559, R560, R561, R562, R563, R564: 1k 5%, symbol Device:R
- removed U402, U403, U404: LP5036, Package_DFN_QFN:VQFN-46-1EP_5x6mm_P0.4mm_EP2.8x3.8mm, symbol Driver_LED:LP5036
- added U1: EAST1410RGBW02, SMD_EAST1410RGBW02_EVE, symbol EAST1410RGBW02:EAST1410RGBW02
Other:
- moved on the sheet: C402, D401, D402, D403, D404, D405, D406, D407, D408, D409, D410, D411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

Commit message: Working on files
Parts:
- removed D401, D402, D403, D404, D405, D406, D407, D408, D409, D410, D411, D412: SMLVN6RGB, LED_SMD:LED_ROHM_SMLVN6, symbol LED:SMLVN6RGB
- removed R401, R402, R403, R404, R405, R406, R407, R408, R409, R410, R411, R412, R413, R414, R415, R416, R417, R418, R419, R420, R421, R422, R423, R424, R425, R426, R427, R428, R429, R430, R431, R432, R433, R434, R435, R436: 1k 5%, symbol Device:R
- added C301: 4.7uF 25V, symbol Device:C
- added C302: 100nF 50V, symbol Device:C
- added U303, U304, U305, U306, U307, U308, U309, U310: EAST1410RGBW02, SMD_EAST1410RGBW02_EVE, symbol EAST1410RGBW02:EAST1410RGBW02
- R301: renamed from R437; value R -> 0E 5%
- R302: renamed from R438; value R -> 0E 5%
- renumbered C402 to C303, R441 to R303, U401 to U301, U1 to U302
Connections:
- net +5V: now also U301.40 (VCC), U302.1, C301.1, C302.1, U303.1, U304.1, U305.1, U306.1, U307.1, U308.1, U309.1, U310.1
- net GND: now also C301.2, C302.2
- net at U301.7 (OUT6): now also U303.4
- net at U301.8 (OUT7): now also U303.5
- net at U301.9 (OUT8): now also U304.2
- net at U301.28 (OUT27): now also U308.5
- net at U301.29 (OUT28): now also U309.2
- net at U301.30 (OUT29): now also U309.3
- net at U301.16 (OUT15): now also U305.5
- net at U301.17 (OUT16): now also U306.2
- net at U301.18 (OUT17): now also U306.3
- net at U301.34 (OUT33): now also U310.3
- net at U301.35 (OUT34): now also U310.4
- net at U301.36 (OUT35): now also U310.5
- net at U301.25 (OUT24): now also U308.2
- net at U301.26 (OUT25): now also U308.3
- net at U301.27 (OUT26): now also U308.4
- net at U301.10 (OUT9): now also U304.3
- net at U301.11 (OUT10): now also U304.4
- net at U301.12 (OUT11): now also U304.5
- net at U301.1 (OUT0): now also U302.2
- net at U301.13 (OUT12): now also U305.2
- net at U301.14 (OUT13): now also U305.3
- net at U301.15 (OUT14): now also U305.4
- net at U301.19 (OUT18): now also U306.4
- net at U301.2 (OUT1): now also U302.3
- net at U301.20 (OUT19): now also U306.5
- net at U301.21 (OUT20): now also U307.2
- net at U301.22 (OUT21): now also U307.3
- net at U301.23 (OUT22): now also U307.4
- net at U301.24 (OUT23): now also U307.5
- net at U301.3 (OUT2): now also U302.4
- net at U301.31 (OUT30): now also U309.4
- net at U301.32 (OUT31): now also U309.5
- net at U301.33 (OUT32): now also U310.2
- net at U301.4 (OUT3): now also U302.5
- net at U301.5 (OUT4): now also U303.2
- net at U301.6 (OUT5): now also U303.3
- no-connect marks 0 -> 9
Other:
- note added: "LED Controller"
- note added: "LED Controller will be place on bottom side of the pcb. Every Diode is current controlled with one channel."
- note added: "LEDs will be place on TOP side of the PCB"
- note added: "Place all decoupling caps as close as the supply pins as possible!"
- title: (none) -> NightLight
- moved on the sheet: C303, R301, R303, U302

Commit message: working on LED PCB
Parts:
- added TP301, TP302, TP303, TP304, TP305, TP306: TestPoint_Small, TestPoint:TestPoint_Loop_D1.80mm_Drill1.0mm_Beaded, symbol Connector:TestPoint_Small
- C301, C302, C303: footprint (none) -> Capacitor_SMD:C_0402_1005Metric_Pad0.74x0.62mm_HandSolder
- R301, R302, R303: footprint (none) -> Resistor_SMD:R_0402_1005Metric_Pad0.72x0.64mm_HandSolder
- U302, U303, U304, U305, U306, U307, U308, U309, U310: footprint SMD_EAST1410RGBW02_EVE -> EAST1410RGBW02:SMD_EAST1410RGBW02_EVE
Connections:
- net +5V: now also TP305.1
- net GND: now also TP304.1, TP306.1
- net LP_EN: now also TP301.1
- net LP_SCL: now also TP302.1
- net LP_SDA: now also TP303.1

Commit message: Finisched digital one
Parts:
- removed R301, R302: 0E 5%, Resistor_SMD:R_0402_1005Metric_Pad0.72x0.64mm_HandSolder, symbol Device:R
- removed R303: 10k 5%, Resistor_SMD:R_0402_1005Metric_Pad0.72x0.64mm_HandSolder, symbol Device:R
- removed U301: LP5036, Package_DFN_QFN:VQFN-46-1EP_5x6mm_P0.4mm_EP2.8x3.8mm, symbol Driver_LED:LP5036
- removed U302, U303, U304, U305, U306, U307, U308, U309, U310: EAST1410RGBW02, EAST1410RGBW02:SMD_EAST1410RGBW02_EVE, symbol EAST1410RGBW02:EAST1410RGBW02
- added C304, C305, C306, C307, C308, C309, C310: C, Capacitor_SMD:C_0402_1005Metric_Pad0.74x0.62mm_HandSolder, symbol Device:C
- added D301, D302, D303, D304, D305, D306, D307, D308, D309, D310: SK6805, LED_SMD:LED_SK6805_PLCC4_2.4x2.7mm_P1.3mm, symbol LED:SK6805
- C301: value 4.7uF 25V -> C
- C302: value 100nF 50V -> C
- C303: value 1uF 50V -> C
Connections:
- net LP_EN is gone; now on net GND: TP301.1
- net LP_SCL is gone; now on net +5V: TP302.1
- net LP_SDA is gone; now on net GND: TP303.1
- net +5V: now also C303.1, TP304.1, C304.1, C305.1, C306.1, C307.1, C308.1, C309.1, C310.1, D301.4 (VDD), D302.4 (VDD), D303.4 (VDD), D304.4 (VDD), D305.4 (VDD), D306.4 (VDD), D307.4 (VDD), D308.4 (VDD), D309.4 (VDD), D310.4 (VDD); no longer TP305.1
- net GND: now also C304.2, C305.2, C306.2, C307.2, C308.2, C309.2, C310.2, D301.2 (VSS), D302.2 (VSS), D303.2 (VSS), D304.2 (VSS), D305.2 (VSS), D306.2 (VSS), D307.2 (VSS), D308.2 (VSS), D309.2 (VSS), D310.2 (VSS); no longer TP304.1, TP306.1
- new net DIN: D301.3 (DIN), TP306.1
- new net DO1: D301.1 (DOUT), D302.3 (DIN)
- new net DO2: D302.1 (DOUT), D303.3 (DIN)
- new net DO3: D303.1 (DOUT), D304.3 (DIN)
- new net DO4: D304.1 (DOUT), D305.3 (DIN)
- new net DO5: D305.1 (DOUT), D306.3 (DIN)
- new net DO6: D306.1 (DOUT), D307.3 (DIN)
- new net DO7: D307.1 (DOUT), D308.3 (DIN)
- new net DO8: D308.1 (DOUT), D309.3 (DIN)
- new net DO9: D309.1 (DOUT), D310.3 (DIN)
- new net DOUT: D310.1 (DOUT), TP305.1
- no-connect marks 9 -> 0
Other:
- note removed: "LED Controller"
- note removed: "LED Controller will be place on bottom side of the pcb. Every Diode is current controlled with one channel."
- note removed: "LEDs will be place on TOP side of the PCB"
- note removed: "Place all decoupling caps as close as the supply pins as possible!"
