File: NightController/usb.kicad_sch (KiCad schematic)
At the start: 0 parts

Commit message: Add parts
Parts:
- added C501: 100nF 50V, symbol Device:C
- added C502, C503, C504, C505: 2.2uF 50V, symbol Device:C
- added J501: USB_C_Receptacle_USB2.0_16P, symbol Connector:USB_C_Receptacle_USB2.0_16P
- added L501, L502: L_Ferrite, symbol Device:L_Ferrite
- added R501, R502: 5.1k 5%, symbol Device:R
- added U501: USBLC6-2P6, Package_TO_SOT_SMD:SOT-666, symbol Power_Protection:USBLC6-2P6
Connections:
- new net GND: C501.2, C502.2, C503.2, C504.2, C505.2, J501.A1 (GND), J501.A12 (GND), J501.B1 (GND), J501.B12 (GND), J501.S1 (SHIELD), R501.2, R502.2, U501.2 (GND)
- new net USBC_D_N: J501.A7 (D-), J501.B7 (D-), U501.1 (I/O1)
- new net USBC_D_P: J501.A6 (D+), J501.B6 (D+), U501.3 (I/O2)
- new net USB_CC1: J501.A5 (CC1), R502.1
- new net USB_CC2: J501.B5 (CC2), R501.1
- new net USB_D_N: U501.6 (I/O1)
- new net USB_D_P: U501.4 (I/O2)
- new net VBUS: C501.1, C502.1, C504.1, J501.A4 (VBUS), J501.A9 (VBUS), J501.B4 (VBUS), J501.B9 (VBUS), L501.1, L502.1, U501.5 (VBUS)
- new net VCC: C503.1, C505.1, L501.2, L502.2
- no-connect marks 0 -> 2

Commit message: Working on schematic
Parts:
- added C506: 0.1u, Capacitor_SMD:C_0603_1608Metric, symbol Device:C_Small
- added FB501: >1A, Inductor_SMD:L_0603_1608Metric, symbol Device:Ferrite_Bead_Small
Connections:
- net GND: now also C506.1, FB501.2; no longer J501.S1 (SHIELD)
- new net: C506.2, FB501.1, J501.S1 (SHIELD)
