File: NightController/Esp32.kicad_sch (KiCad schematic)
At the start: 0 parts

Commit message: Add parts
Parts:
- added U401: ESP32-S2-WROVER, RF_Module:ESP32-S2-WROVER, symbol RF_Module:ESP32-S2-WROVER
Connections:
- new net +3.3V: U401.2 (3V3)
- new net GND: U401.1 (GND), U401.26 (GND), U401.42 (GND), U401.43 (GND)

Commit message: Working on schematic
Parts:
- added C401, C402, C403: 0.1u, Capacitor_SMD:C_0603_1608Metric, symbol Device:C_Small
- added R401: 10k, Resistor_SMD:R_0603_1608Metric, symbol Device:R_Small
- added SW401: Reset, ESP32-S2-Breakout:Alps_SKRK, symbol Switch:SW_Push
- added SW402: Boot, ESP32-S2-Breakout:Alps_SKRK, symbol Switch:SW_Push
Connections:
- net GND: now also C401.2, C402.2, C403.2, SW401.1, SW402.1
- net at U401.41 (EN): now also C403.1, R401.2
- new net +3V3: R401.1
- new net EN: C401.1, SW401.2
- new net IO0: C402.1, SW402.2
Other:
- note added: "Boot/Reset Switches"

Commit message: update schematic
Parts:
- added C404: C, Capacitor_SMD:C_0402_1005Metric_Pad0.74x0.62mm_HandSolder, symbol Device:C
- added C405: 100nF 50V, Capacitor_SMD:C_0402_1005Metric_Pad0.74x0.62mm_HandSolder, symbol Device:C
- added C406: 4.7uF 50V, Capacitor_SMD:C_0603_1608Metric, symbol Device:C_Small
- added C407: 220nF 50V, Capacitor_SMD:C_0603_1608Metric, symbol Device:C_Small
- added D401: SK6805, LED_SMD:LED_SK6805_PLCC4_2.4x2.7mm_P1.3mm, symbol LED:SK6805
- added J401: Conn_01x06_Socket, symbol Connector:Conn_01x06_Socket
- added Q401, Q402: BC817W, Package_TO_SOT_SMD:SOT-323_SC-70, symbol Transistor_BJT:BC817W
- added R402, R403: 10k, Resistor_SMD:R_0603_1608Metric, symbol Device:R_Small
- added TP401, TP402, TP403: TestPoint_Small, TestPoint:TestPoint_Loop_D1.80mm_Drill1.0mm_Beaded, symbol Connector:TestPoint_Small
- C403: value 0.1u -> 1uF 50V
Connections:
- net EN is gone; now on net CHIP_PU: C401.1, SW401.2
- net +3.3V: now also C405.2, C406.2, C407.2, J401.1 (Pin_1)
- net GND: now also C404.2, C405.1, C406.1, C407.1, D401.2 (VSS), J401.6 (Pin_6), TP403.1
- net CHIP_PU: now reaches C403.1, R401.2, U401.41 (EN)
- net CHIP_PU: now also Q401.3 (C)
- net ESP_TX: now reaches U401.20 (IO17)
- net RGB_LED: now reaches U401.21 (IO18)
- net RGB_LED: now also D401.3 (DIN), TP401.1
- net ESP_RTS: now reaches U401.22 (USB_D-)
- net ESP_CTS: now reaches U401.23 (USB_D+)
- net ESP_RX: now reaches U401.24 (IO21)
- net GPIO0: now reaches U401.3 (IO00)
- net GPIO0: now also Q402.3 (C)
- net TXD0: now reaches U401.37 (TXD0)
- net TXD0: now also J401.3 (Pin_3)
- net RXD0: now reaches U401.38 (RXD0)
- net RXD0: now also J401.2 (Pin_2)
- new net: Q402.1 (B), R403.2
- new net: Q401.1 (B), R402.2
- new net +VSYS: C404.1, D401.4 (VDD), TP402.1
- new net DO1: D401.1 (DOUT)
- new net DTR: J401.4 (Pin_4), Q402.2 (E), R402.1
- new net RTS: J401.5 (Pin_5), Q401.2 (E), R403.1
- no-connect marks 0 -> 29
Other:
- note added: "Auto Programming circuit"
- note added: "Decoupling caps"
- note added: "ESP32-S2 WiFi Module"
- note added: "Programming connector"
- note added: "RGB LED"
- moved on the sheet: C403, R401
