File: NightController/daughter_board.kicad_sch (KiCad schematic)
At the start: 0 parts

Commit message: Add parts
Parts:
- added J301, J302: Conn_02x20_Odd_Even, Connector_Molex:Molex_SlimStack_54722-0404_2x20_P0.50mm_Vertical, symbol Connector_Generic:Conn_02x20_Odd_Even
Connections:
- new net +3V3: J301.2 (Pin_2), J301.37 (Pin_37), J301.39 (Pin_39), J301.4 (Pin_4), J302.2 (Pin_2), J302.37 (Pin_37), J302.39 (Pin_39), J302.4 (Pin_4)
- new net +5V: J301.32 (Pin_32), J301.34 (Pin_34), J301.7 (Pin_7), J301.9 (Pin_9), J302.32 (Pin_32), J302.34 (Pin_34), J302.7 (Pin_7), J302.9 (Pin_9)
- new net DIN: J302.29 (Pin_29)
- new net DOUT: J302.27 (Pin_27)
- new net GND: J301.1 (Pin_1), J301.10 (Pin_10), J301.3 (Pin_3), J301.31 (Pin_31), J301.33 (Pin_33), J301.35 (Pin_35), J301.36 (Pin_36), J301.38 (Pin_38), J301.40 (Pin_40), J301.5 (Pin_5), J301.6 (Pin_6), J301.8 (Pin_8), J302.1 (Pin_1), J302.10 (Pin_10), J302.3 (Pin_3), J302.31 (Pin_31), J302.33 (Pin_33), J302.35 (Pin_35), J302.36 (Pin_36), J302.38 (Pin_38), J302.40 (Pin_40), J302.5 (Pin_5), J302.6 (Pin_6), J302.8 (Pin_8)
- no-connect marks 0 -> 38
Other:
- note added: "Connectors to Controller board"

Commit message: update schematic
Connections:
- net +5V renamed +VSYS
Changed lines of the file:
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@@
 			)
 		)
-		(property "Value" "+5V"
+		(property "Value" "+VSYS"
 			(at 72.39 71.1201 90)
 			(effects
@@
 			)
 		)
-		(property "Value" "+5V"
+		(property "Value" "+VSYS"
 			(at 194.31 104.1399 90)
 			(effects
@@
 			)
 		)
-		(property "Value" "+5V"
+		(property "Value" "+VSYS"
 			(at 148.59 71.1201 90)
 			(effects
@@
 			)
 		)
-		(property "Value" "+5V"
+		(property "Value" "+VSYS"
 			(at 118.11 104.1399 90)
 			(effects

Commit message: Add Right Connector
Parts:
- J301, J302: footprint Connector_Molex:Molex_SlimStack_54722-0404_2x20_P0.50mm_Vertical -> Connector_Molex:Molex_SlimStack_55560-0401_2x20_P0.50mm_Vertical
Changed lines of the file:
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@@
 			)
 		)
-		(property "Footprint" "Connector_Molex:Molex_SlimStack_54722-0404_2x20_P0.50mm_Vertical"
+		(property "Footprint" "Connector_Molex:Molex_SlimStack_55560-0401_2x20_P0.50mm_Vertical"
 			(at 93.98 86.36 0)
 			(effects
@@
 			)
 		)
-		(property "Footprint" "Connector_Molex:Molex_SlimStack_54722-0404_2x20_P0.50mm_Vertical"
+		(property "Footprint" "Connector_Molex:Molex_SlimStack_55560-0401_2x20_P0.50mm_Vertical"
 			(at 170.18 86.36 0)
 			(effects
